File: BD0004.brd (EAGLE design)
At the start: 67.3 x 39.4 mm, 30 parts, among them J1 HEADER_1X3MALE, J2 HEADER_1X3FEMALE, J3 1050171001, J4 20021121-00010C4LF, U1 ATSAMD11D14A-MNT, U2 AP2114H-3.3TRG1, X1 MC-146-32.7680JKA-A0:ROHS

Commit message: initial updates from v1. (not sure what was changed)
Parts:
- removed CR1: USBLC6-2P6SOT-666-M, Clock:SOT-666-M
- B1: device Clock:4-SMD_BUTTON -> DroidForge:4-SMD_BUTTON
- C1, C2, C3, C6, C7, C8: device adafruit:C0402 -> DroidForge:0402
- C4, C5: device adafruit:C0805 -> DroidForge:0402
- J1: device Clock:M3SMD -> DroidForge:M3SMD_RIGHTANGLE
- J2: device Clock:F3SMD -> DroidForge:F3SMD_RIGHTANGLE
- J3: value 1050171001 -> CONN_MICROUSB_FEMALE; device Clock:CON00679_5 -> DroidForge:CON00679_5
- J4: value 20021121-00010C4LF -> CORTEX-M_DEBUG_HEADER; device Clock:CONN_00010C4LF -> DroidForge:CONN_00010C4LF
- L1, L2, L3: value WS2812B -> WS2812B-B; device Clock:SK6812 -> DroidForge:SK6812-B
- R1: device adafruit:R0402 -> DroidForge:0402
- TP1, TP2, TP3, TP4, TP5, TP6, TP7, TP8, TP9: device Clock:R-1-CR -> DroidForge:R-1-CR
- U1: value ATSAMD11D14A-MNT -> SAMD11D14A; device Clock:QFN24_4X4MC -> DroidForge:QFN24_4X4MC
- U2: device Clock:SOT-223 -> DroidForge:SOT-223
- X1: device Clock:4-SMD_FLAT_LEADS -> DroidForge:4-SMD_FLAT_LEADS
Connections:
- removed net N$1: CR1.3, J3.3
- removed net N$3: CR1.1, J3.2
- removed net USB_D+: CR1.4, U1.22
- removed net USB_D-: CR1.6, U1.21
- new net D+: J3.3, U1.22
- new net D-: J3.2, U1.21
- net GND: now also C1.P$2, C2.P$2, C3.P$2, C4.P$2, C5.P$2, C6.P$2, C7.P$2, C8.P$2; no longer C1.2, C2.2, C3.2, C4.2, C5.2, C6.2, C7.2, C8.2, CR1.2
- net N$4: now also C6.P$1; no longer C6.1
- net N$5: now also C7.P$1; no longer C7.1
- net RESET: now also R1.P$1; no longer R1.1
- net VCC: now also C1.P$1, C2.P$1, C3.P$1, C5.P$1, C8.P$1, R1.P$2, U2.4; no longer C1.1, C2.1, C3.1, C5.1, C8.1, CR1.5, R1.2
- net VIN: now also C4.P$1; no longer C4.1
Routing:
- net VCC: track 176.5 -> 195.6 mm, vias 5 -> 2
- net D+: track 0.00 -> 8.15 mm
- net D-: track 0.00 -> 8.11 mm
- net USB_D+: track 3.20 -> 0.00 mm
- net USB_D-: track 3.20 -> 0.00 mm
- net N$3: track 3.05 -> 0.00 mm
- net N$1: track 2.99 -> 0.00 mm
