File: BD0004.sch (EAGLE design)
At the start: 30 parts, among them J1 HEADER_1X3MALE, J2 HEADER_1X3FEMALE, J3 1050171001, J4 20021121-00010C4LF, U1 ATSAMD11D14A-MNT, U2 AP2114H-3.3TRG1, X1 MC-146-32.7680JKA-A0:ROHS

Commit message: initial updates from v1. (not sure what was changed)
Parts:
- removed CR1: USBLC6-2P6SOT-666-M, Clock:USBLC6-2P6SOT-666-M
- B1: device Clock:EVQ-P7A01P -> DroidForge:EVQ-P7A01P
- C1, C2, C3, C6, C7, C8: device adafruit:C-USC0402 -> DroidForge:CAPACITOR-0402
- C4, C5: device adafruit:C-USC0805 -> DroidForge:CAPACITOR-0402
- J1: device Clock:HEADER_1X3MALE -> DroidForge:HEADER_1X3MALE
- J2: device Clock:HEADER_1X3FEMALE -> DroidForge:HEADER_1X3FEMALE
- J3: value 1050171001 -> CONN_MICROUSB_FEMALE; device Clock:1050171001 -> DroidForge:CONN_MICROUSB_FEMALE
- J4: value 20021121-00010C4LF -> CORTEX-M_DEBUG_HEADER; device Clock:20021121-00010C4LF -> DroidForge:CORTEX-M_DEBUG_HEADER
- L1, L2, L3: value WS2812B -> WS2812B-B; device Clock:WS2812B -> DroidForge:WS2812B-B
- R1: device adafruit:R-US_R0402 -> DroidForge:RESISTOR-0402
- TP1, TP2, TP3, TP4, TP5, TP6, TP7, TP8, TP9: device Clock:POGO -> DroidForge:POGO
- U1: value ATSAMD11D14A-MNT -> SAMD11D14A; device Clock:ATSAMD11D14A-MNT -> DroidForge:SAMD11D14A
- U2: device Clock:AP2114H-3.3TRG1 -> DroidForge:AP2114H-3.3TRG1
- X1: device Clock:MC-146-32.7680JKA-A0:ROHS -> DroidForge:MC-146-32.7680JKA-A0:ROHS
Connections:
- removed net N$1: CR1.I/O2_2, J3.3
- removed net N$3: CR1.I/O1_2, J3.2
- removed net USB_D+: CR1.I/O1, U1.PA25
- removed net USB_D-: CR1.I/O2, U1.PA24
- new net D+: J3.D+, U1.PA25
- new net D-: J3.D-, U1.PA24
- net GND: now also J3.GND; no longer CR1.GND, J3.5
- net VCC: now also U2.VOUT; no longer CR1.VBUS
- net VIN: now also J3.5V; no longer J3.1
Other:
- moved on the sheet: B1, C1, C2, C4, C5, C8, L1, L2, L3, U2
