File: BD0006.brd (EAGLE design)
At the start: 67.3 x 33 mm, 47 parts, among them J1 HEADER_1X3MALE, J2 HEADER_1X3FEMALE

Commit message: initial updates from v1. (not sure what was changed)
Parts:
- C1, C10, C11, C12, C13, C14, C15, C16, C17, C18, C19, C2, C20, C3, C4, C5, C6, C7, C8+, C9: device adafruit:C0402 -> DroidForge:0402
- J1: device Clock:M3SMD -> DroidForge:M3SMD_RIGHTANGLE
- J2: device Clock:F3SMD -> DroidForge:F3SMD_RIGHTANGLE
- JP2: value HEADER_1X4S -> HEADER_1X4; device Clock:1X04 -> DroidForge:1X04-CLEANBIG
- L1, L10, L11, L12, L13, L14, L15, L16, L17, L18, L19, L2, L20, L3, L4, L5, L6, L7, L8, L9: value WS2812B -> WS2812B-B; device Clock:SK6812 -> DroidForge:SK6812-B
- TP1, TP2, TP3, TP4: device Clock:TEST_POINT -> DroidForge:TEST_POINT
Connections:
- net GND: now also C1.P$2, C10.P$2, C11.P$2, C12.P$2, C13.P$2, C14.P$2, C15.P$2, C16.P$2, C17.P$2, C18.P$2, C19.P$2, C2.P$2, C20.P$2, C3.P$2, C4.P$2, C5.P$2, C6.P$2, C7.P$2, C8+.P$2, C9.P$2; no longer C1.2, C10.2, C11.2, C12.2, C13.2, C14.2, C15.2, C16.2, C17.2, C18.2, C19.2, C2.2, C20.2, C3.2, C4.2, C5.2, C6.2, C7.2, C8+.2, C9.2
- net VCC: now also C1.P$1, C10.P$1, C11.P$1, C12.P$1, C13.P$1, C14.P$1, C15.P$1, C16.P$1, C17.P$1, C18.P$1, C19.P$1, C2.P$1, C20.P$1, C3.P$1, C4.P$1, C5.P$1, C6.P$1, C7.P$1, C8+.P$1, C9.P$1; no longer C1.1, C10.1, C11.1, C12.1, C13.1, C14.1, C15.1, C16.1, C17.1, C18.1, C19.1, C2.1, C20.1, C3.1, C4.1, C5.1, C6.1, C7.1, C8+.1, C9.1
Routing:
- net VCC: track 342.4 -> 345.4 mm
- net DIN: track 73.5 -> 74.2 mm
