File: BD0006.sch (EAGLE design)
At the start: 47 parts, among them J1 HEADER_1X3MALE, J2 HEADER_1X3FEMALE

Commit message: initial updates from v1. (not sure what was changed)
Parts:
- C1, C10, C11, C12, C13, C14, C15, C16, C17, C18, C19, C2, C20, C3, C4, C5, C6, C7, C8+, C9: device adafruit:C-USC0402 -> DroidForge:CAPACITOR-0402
- J1: device Clock:HEADER_1X3MALE -> DroidForge:HEADER_1X3MALE
- J2: device Clock:HEADER_1X3FEMALE -> DroidForge:HEADER_1X3FEMALE
- JP2: value HEADER_1X4S -> HEADER_1X4; device Clock:HEADER_1X4S -> DroidForge:HEADER_1X4
- L1, L10, L11, L12, L13, L14, L15, L16, L17, L18, L19, L2, L20, L3, L4, L5, L6, L7, L8, L9: value WS2812B -> WS2812B-B; device Clock:WS2812B -> DroidForge:WS2812B-B
- TP1, TP2, TP3, TP4: device Clock:TEST_POINT -> DroidForge:TEST_POINT
Other:
- moved on the sheet: C1, C10, C11, C12, C13, C14, C15, C16, C17, C18, C19, C2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
