File: BD0007.brd (EAGLE design)
At the start: 19.1 x 33 mm, 17 parts, among them J1 HEADER_1X3MALE, J2 HEADER_1X3FEMALE

Commit message: initial updates from v1. (not sure what was changed)
Parts:
- C1, C2, C3, C4, C5: device adafruit:C0402 -> DroidForge:0402
- J1: device Clock:M3SMD -> DroidForge:M3SMD_RIGHTANGLE
- J2: device Clock:F3SMD -> DroidForge:F3SMD_RIGHTANGLE
- JP1: value HEADER_1X4S -> HEADER_1X4; device Clock:1X04 -> DroidForge:1X04-CLEANBIG
- L1, L2, L3, L4, L5: value WS2812B -> WS2812B-B; device Clock:SK6812 -> DroidForge:SK6812-B
- TP1, TP2, TP3, TP4: device Clock:TEST_POINT -> DroidForge:TEST_POINT
Connections:
- net GND: now also C1.P$2, C2.P$2, C3.P$2, C4.P$2, C5.P$2; no longer C1.2, C2.2, C3.2, C4.2, C5.2
- net VCC: now also C1.P$1, C2.P$1, C3.P$1, C4.P$1, C5.P$1; no longer C1.1, C2.1, C3.1, C4.1, C5.1
Routing:
- net VCC: track 82.8 -> 83.9 mm
- net DIN: track 39.8 -> 39.2 mm
- net DOUT: track 50.9 -> 50.4 mm
