File: BD0008.brd (EAGLE design)
At the start: 19.1 x 33 mm, 9 parts, among them J1 HEADER_1X3MALE, J2 HEADER_1X3FEMALE

Commit message: initial updates from v1. (not sure what was changed)
Parts:
- C1: device adafruit:C0402 -> DroidForge:0402
- J1: device Clock:M3SMD -> DroidForge:M3SMD_RIGHTANGLE
- J2: device Clock:F3SMD -> DroidForge:F3SMD_RIGHTANGLE
- JP1: value HEADER_1X4S -> HEADER_1X4; device Clock:1X04 -> DroidForge:1X04-CLEANBIG
- L1: value WS2812B -> WS2812B-B; device Clock:SK6812 -> DroidForge:SK6812-B
- TP1, TP2, TP3, TP4: device Clock:TEST_POINT -> DroidForge:TEST_POINT
Connections:
- net GND: now also C1.P$2; no longer C1.2
- net VCC: now also C1.P$1; no longer C1.1
Routing:
- net VCC: track 64.9 -> 65.6 mm
- net DIN: track 36.9 -> 36.4 mm
- net DOUT: track 51.8 -> 51.3 mm
