File: BD0005.sch (EAGLE design)
At the start: 68 parts, among them J1 1050171001, J3 HEADER_1X3FEMALE, J4 HEADER_1X3FEMALE, U1 ATSAMD11D14A-MNT, U2 AP2114H-3.3TRG1, X1 MC-146-32.7680JKA-A0:ROHS

Commit message: initial updates from v1. (not sure what was changed)
Parts:
- removed CR1: USBLC6-2P6SOT-666-M, Clock:USBLC6-2P6SOT-666-M
- removed JP2: (no value), adafruit:PINHD-1X3
- added J2: HEADER_1X3, DroidForge:HEADER_1X3
- B1, B2: device Clock:EVQ-P7A01P -> DroidForge:EVQ-P7A01P
- C1, C2: device adafruit:C-USC0805 -> DroidForge:CAPACITOR-0402
- C10, C11, C12, C13, C14, C15, C16, C17, C18, C19, C20, C21, C22, C23, C24, C25, C3, C4, C5, C6, C7, C8, C9: device adafruit:C-USC0402 -> DroidForge:CAPACITOR-0402
- J1: value 1050171001 -> CONN_MICROUSB_FEMALE; device Clock:1050171001 -> DroidForge:CONN_MICROUSB_FEMALE
- J3, J4: device Clock:HEADER_1X3FEMALE -> DroidForge:HEADER_1X3FEMALE
- JP1: value PINHD-1X10 -> HEADER_1X10; device adafruit:PINHD-1X10 -> DroidForge:HEADER_1X10
- L1, L10, L11, L12, L13, L14, L15, L16, L17, L18, L19, L2, L20, L3, L4, L5, L6, L7, L8, L9: value WS2812B -> WS2812B-B; device Clock:WS2812B -> DroidForge:WS2812B-B
- R1, R3: device adafruit:R-US_R0402 -> DroidForge:RESISTOR-0402
- R2: value 3352T-1-104LF -> POT_THUMBWHEEL_3352T-1-104LF; device Clock:3352T-1-104LF -> DroidForge:POT_THUMBWHEEL_3352T-1-104LF
- TP1, TP2, TP3, TP4, TP5, TP6, TP7, TP8, TP9: device Clock:TEST_POINT -> DroidForge:TEST_POINT
- U1: value ATSAMD11D14A-MNT -> SAMD11D14A; device Clock:ATSAMD11D14A-MNT -> DroidForge:SAMD11D14A
- U2: device Clock:AP2114H-3.3TRG1 -> DroidForge:AP2114H-3.3TRG1
- X1: device Clock:MC-146-32.7680JKA-A0:ROHS -> DroidForge:MC-146-32.7680JKA-A0:ROHS
Connections:
- removed net N$1: CR1.I/O2_2, J1.3
- removed net N$3: CR1.I/O1_2, J1.2
- net GND: now also J1.GND, J2.P$2; no longer CR1.GND, J1.5, JP2.2
- net USB_D+: now also J1.D+; no longer CR1.I/O1
- net USB_D-: now also J1.D-; no longer CR1.I/O2
- net VCC: now also J2.P$1, U2.VOUT; no longer CR1.VBUS, JP2.1
- net VIN: now also J1.5V, J2.P$3; no longer J1.1, JP2.3
Other:
- moved on the sheet: C1, C10, C11, C12, C13, C14, C15, C16, C17, C18, C19, C2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

Commit message: changed SAMD11 to SAMD21E (in process)
Parts:
- removed U1: SAMD11D14A, DroidForge:SAMD11D14A
- added U3: SAMD21E__A-MU_16(64K), DroidForge:SAMD21E__A-MU_16(64K)
- B1, B2: value EVQ-P7A01P -> SWITCH_EVQ-P7A01P; device DroidForge:EVQ-P7A01P -> DroidForge:SWITCH_EVQ-P7A01P
- U2: value AP2114H-3.3TRG1 -> REG_AP2114H-3.3TRG1; device DroidForge:AP2114H-3.3TRG1 -> DroidForge:REG_AP2114H-3.3TRG1
- X1: value MC-146-32.7680JKA-A0:ROHS -> XTAL_MC-146-32.7680JKA-A0:ROHS; device DroidForge:MC-146-32.7680JKA-A0:ROHS -> DroidForge:XTAL_MC-146-32.7680JKA-A0:ROHS
Connections:
- removed net USB_D+: J1.D+, U1.PA25
- removed net USB_D-: J1.D-, U1.PA24
- new net A10: U3.PA10
- new net A11: U3.PA11
- new net A16: U3.PA16
- new net A17: U3.PA17
- new net A18: U3.PA18
- new net A19: U3.PA19
- new net A22: U3.PA22
- new net A23: U3.PA23
- new net A24: U3.PA24
- new net A25: U3.PA25
- new net A27: U3.PA27
- new net A28: U3.PA28
- new net A30: U3.PA30
- new net A31: U3.PA31
- new net A8: U3.PA08
- new net A9: U3.PA09
- new net D+: J1.D+
- new net D-: J1.D-
- net A2: now also U3.PA02; no longer U1.PA02
- net A3: now also U3.PA03; no longer U1.PA03
- net A4: now also U3.PA04; no longer U1.PA04
- net A5: now also U3.PA05; no longer U1.PA05
- net A6: now also U3.PA06; no longer U1.PA06
- net A7: now also U3.PA07; no longer U1.PA07
- net BIN: no longer U1.PA17
- net DIN: no longer U1.PA27
- net DOUT_1: no longer U1.PA15
- net DOUT_2: no longer U1.PA16
- net GND: now also U3.EPAD, U3.GND, U3.GND_2; no longer C3.2, U1.EPAD, U1.GND
- net MISO: no longer U1.PA14
- net MOSI: no longer U1.PA10
- net N$4: now also U3.PA00; no longer U1.PA08
- net N$5: now also U3.PA01; no longer U1.PA09
- net RESET: no longer U1.PA28/!RST
- net SCK: no longer U1.PA11
- net SCL: no longer U1.PA23
- net SDA: no longer U1.PA22
- net SWCLK: no longer U1.PA30
- net SWDIO: no longer U1.PA31
- net VCC: no longer C3.1, U1.VDDIO/IN/ANA
Other:
- note added: "D+"
- note added: "D-"
- note added: "DOUT_1"
- note added: "MISO"
- note added: "MOSI"
- note added: "SCK"
- note added: "SCL"
- note added: "SDA"
- note added: "SWCLK"
- note added: "SWDIO"
- moved on the sheet: B1, B2, C1, C10, C11, C12, C13, C14, C15, C16, C17, C18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
