File: BD0005 (main)/BD0005.sch (EAGLE design)
At the start: 67 parts, among them J1 CONN_MICROUSB_FEMALE, J2 HEADER_1X3, J3 HEADER_1X3FEMALE, J4 HEADER_1X3FEMALE, U2 REG_AP2114H-3.3TRG1, U3 SAMD21E__A-MU_16(64K), X1 XTAL_MC-146-32.7680JKA-A0:ROHS

Commit message: Placed new microcontroller on pcb
Parts:
- added C26, C27: 0.1uF, DroidForge:CAPACITOR-0402
Connections:
- removed net A10: U3.PA10
- removed net A11: U3.PA11
- removed net A16: U3.PA16
- removed net A17: U3.PA17
- removed net A18: U3.PA18
- removed net A19: U3.PA19
- removed net A22: U3.PA22
- removed net A24: U3.PA24
- removed net A25: U3.PA25
- removed net A30: U3.PA30
- removed net A31: U3.PA31
- removed net A8: U3.PA08
- removed net A9: U3.PA09
- new net N$2: C3.1, U3.VDDIN
- new net N$3: C26.1, U3.VDDANA
- new net N$6: C27.1, U3.VDDCORE
- net BIN: now also U3.PA11
- net D+: now also U3.PA25
- net D-: now also U3.PA24
- net DIN: now also U3.PA08
- net DOUT_1: now also U3.PA09
- net DOUT_2: now also U3.PA10
- net GND: now also C26.2, C27.2, C3.2
- net MISO: now also U3.PA22
- net MOSI: now also U3.PA18
- net RESET: now also U3.!RESET
- net SCK: now also U3.PA19
- net SCL: now also U3.PA17
- net SDA: now also U3.PA16
- net SWCLK: now also U3.PA30
- net SWDIO: now also U3.PA31
Other:
- note removed: "DOUT_1"
- moved on the sheet: B1, B2, C3, R1, R2, R3

Commit message: Finished rerouting board for new SAMD21E processor. Also added VCC connection to processor on schematic
Connections:
- removed net N$2: C3.1, U3.VDDIN
- removed net N$3: C26.1, U3.VDDANA
- net VCC: now also C26.1, C3.1, U3.VDDANA, U3.VDDIN
Changed lines of the file:
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@@
 <part name="C27" library="DroidForge" library_urn="urn:adsk.eagle:library:16489927" deviceset="CAPACITOR" device="-0402" package3d_urn="urn:adsk.eagle:package:16500214/3" value="0.1uF"/>
 <part name="GND14" library="DroidForge" library_urn="urn:adsk.eagle:library:16489927" deviceset="GND" device="" value="GND"/>
+<part name="SUPPLY6" library="DroidForge" library_urn="urn:adsk.eagle:library:16489927" deviceset="VCC" device=""/>
 </parts>
 <sheets>
@@
 </instance>
 <instance part="GND14" gate="G$1" x="-20.32" y="-48.26" smashed="yes"/>
+<instance part="SUPPLY6" gate="G$1" x="-27.94" y="-27.94" smashed="yes">
+<attribute name="VALUE" x="-30.48" y="-27.178" size="1.778" layer="96"/>
+</instance>
 </instances>
 <busses>
@@
 <wire x1="33.02" y1="25.4" x2="33.02" y2="27.94" width="0.1524" layer="91"/>
 </segment>
+<segment>
+<pinref part="C3" gate="G$1" pin="1"/>
+<pinref part="U3" gate="A" pin="VDDIN"/>
+<wire x1="-30.48" y1="-35.56" x2="-30.48" y2="-30.48" width="0.1524" layer="91"/>
+<wire x1="-30.48" y1="-30.48" x2="-27.94" y2="-30.48" width="0.1524" layer="91"/>
+<pinref part="SUPPLY6" gate="G$1" pin="VCC"/>
+<wire x1="-27.94" y1="-30.48" x2="-15.24" y2="-30.48" width="0.1524" layer="91"/>
+<junction x="-27.94" y="-30.48"/>
+<pinref part="C26" gate="G$1" pin="1"/>
+<wire x1="-20.32" y1="-35.56" x2="-20.32" y2="-33.02" width="0.1524" layer="91"/>
+<wire x1="-20.32" y1="-33.02" x2="-12.7" y2="-33.02" width="0.1524" layer="91"/>
+<pinref part="U3" gate="A" pin="VDDANA"/>
+<wire x1="-12.7" y1="-33.02" x2="-12.7" y2="-30.48" width="0.1524" layer="91"/>
+<wire x1="-20.32" y1="-33.02" x2="-27.94" y2="-33.02" width="0.1524" layer="91"/>
+<wire x1="-27.94" y1="-33.02" x2="-27.94" y2="-30.48" width="0.1524" layer="91"/>
+<junction x="-20.32" y="-33.02"/>
+</segment>
 </net>
 <net name="VIN" class="0">
@@
 </segment>
 </net>
-<net name="N$2" class="0">
-<segment>
-<pinref part="C3" gate="G$1" pin="1"/>
-<pinref part="U3" gate="A" pin="VDDIN"/>
-<wire x1="-30.48" y1="-35.56" x2="-30.48" y2="-30.48" width="0.1524" layer="91"/>
-<wire x1="-30.48" y1="-30.48" x2="-15.24" y2="-30.48" width="0.1524" layer="91"/>
-</segment>
-</net>
-<net name="N$3" class="0">
-<segment>
-<pinref part="C26" gate="G$1" pin="1"/>
-<wire x1="-20.32" y1="-35.56" x2="-20.32" y2="-33.02" width="0.1524" layer="91"/>
-<wire x1="-20.32" y1="-33.02" x2="-12.7" y2="-33.02" width="0.1524" layer="91"/>
-<pinref part="U3" gate="A" pin="VDDANA"/>
-<wire x1="-12.7" y1="-33.02" x2="-12.7" y2="-30.48" width="0.1524" layer="91"/>
-</segment>
-</net>
